File: hardware/blaster.kicad_sch (KiCad schematic)
At the start: 16 parts, among them Q201 2N2222, Q202 2N2222, SW201 Slide switch, SW202 Trigger button

Commit message: Redraw schematics on A4 in KiCad colours with larger text
Parts:
- SW202: value Trigger button -> Trigger
Other:
- note added: "(TSAL6100) makes aiming fair."
- note added: "1k limits the base current; 10k holds it off while the XIAO"
- note added: "Button between D0 and GND. No"
- note added: "C (check yours)."
- note added: "D1 sends the 38 kHz coded burst into the base. 22R sets"
- note added: "Flashes on every shot."
- note added: "I2C address 0x3C, 100 kHz. VCC goes on VBAT: the screen"
- note added: "Long leg (+) to 220R."
- note added: "The blaster is also the game host: it runs the CamoBots"
- note added: "The switch sits in the battery + lead. VBAT"
- note added: "battery. Fit the battery and switch last."
- note added: "boots. 10R keeps the speaker current safe. Speaker + goes"
- note added: "fire. Hold 3 s to stop a round."
- note added: "holds D0 HIGH. Press = LOW ="
- note added: "hotspot and the web page. The BOOT button doubles as a spare"
- note added: "is the battery after the switch and goes to"
- note added: "leg (+) of the IR LED goes toward 22R. A narrow-beam LED"
- note added: "resistor: the internal pull-up"
- note added: "stays blank on 3V3. The module has its own I2C pull-"
- note added: "swap VCC and GND. No OLED? The game still runs."
- note added: "the BAT+ pad under the XIAO. Charge through"
- note added: "the LED pulse current (10-15R = longer range). The long"
- note added: "the XIAO USB-C port. The 5V pin is dead on"
- note added: "to VBAT. 2N2222 / S8050: flat face to you, legs down = E B"
- note added: "trigger."
- note added: "ups. Check the pin order printed on yours, some boards"
- note removed: "10R keeps speaker current safe. Speaker + goes to VBAT, not 5V."
- note removed: "1k limits base current; 10k holds it off while the XIAO boots."
- note removed: "22R sets the LED pulse current (10-15R = longer range)."
- note removed: "2N2222 / S8050: flat face to you, legs down = E B C (check yours)."
- note removed: "A narrow-beam LED (TSAL6100) makes aiming fair."
- note removed: "BOOT button doubles as a spare trigger."
- note removed: "Button between D0 and GND."
- note removed: "Charge through the XIAO USB-C port."
- note removed: "Check the pin order printed on yours:"
- note removed: "D1 sends the 38 kHz coded burst into the base."
- note removed: "Fit the battery and switch last."
- note removed: "Flashes on"
- note removed: "Hold 3 s to stop a round."
- note removed: "I2C address 0x3C, 100 kHz."
- note removed: "Long leg (+)"
- note removed: "Long leg (+) of the IR LED goes toward 22R."
- note removed: "No OLED? The game still runs."
- note removed: "No resistor: the XIAO's internal"
- note removed: "Press = LOW = fire."
- note removed: "Switch sits in the battery + lead."
- note removed: "The 5V pin is dead on battery, so"
- note removed: "The blaster is also the game host:"
- note removed: "The module has its own I2C pull-ups."
- note removed: "VBAT = battery after the switch,"
- note removed: "VCC on VBAT: it stays blank on 3V3."
- note removed: "every shot."
- note removed: "it runs the CamoBots hotspot and the web page."
- note removed: "loads that need more than 3.3 V use VBAT."
- note removed: "pull-up holds D0 HIGH."
- note removed: "some boards swap VCC and GND."
- note removed: "to the BAT+ pad under the XIAO."
- note removed: "toward 220R."
