File: hardware/body.kicad_sch (KiCad schematic)
At the start: 17 parts, among them Q101 2N2222, SW101 Slide switch, U102 TSOP38238

Commit message: Redraw schematics on A4 in KiCad colours with larger text
Parts:
- BT101: value LiPo 3.7V 500mAh -> LiPo 500mAh
Other:
- note added: "100R + 4.7u filter its supply. Dome facing you,"
- note added: "1k limits the base current; 10k holds it off while the XIAO"
- note added: "900, covered about 100. Below 40% of"
- note added: "C (check yours)."
- note added: "D0-D5 are ADC1 pins, safe to read with Wi-Fi on. D2 is a boot"
- note added: "More light = lower LDR resistance ="
- note added: "R101 R108 R109"
- note added: "Speaker 8 ohm 1 W (TR-WS-2014B)"
- note added: "The longest leg is the common anode: it goes to 3V3. A"
- note added: "The switch sits in the battery + lead. VBAT"
- note added: "battery. Fit the battery and switch last."
- note added: "boots. 10R keeps the speaker current safe. Speaker + goes"
- note added: "dome."
- note added: "hiding, red = caught, rainbow = survived the round."
- note added: "higher reading on D1. Room light about"
- note added: "is the battery after the switch and goes to"
- note added: "legs down: OUT GND VS. Never paint over the"
- note added: "misbehaves, move the speaker to D8 (GPIO7)."
- note added: "pin driven LOW turns its colour on. Red gets a bigger"
- note added: "resistor because it is brighter. Teal = waiting, blue ="
- note added: "strapping pin: the 10k pull-down keeps it low. If boot"
- note added: "the BAT+ pad under the XIAO. Charge through"
- note added: "the XIAO USB-C port. The 5V pin is dead on"
- note added: "the start level counts as covered."
- note added: "to VBAT. 2N2222 / S8050: flat face to you, legs down = E B"
- note removed: "100R + 4.7u filter its supply."
- note removed: "10R keeps speaker current safe. Speaker + goes to VBAT, not 5V."
- note removed: "1k limits base current; 10k holds it off while the XIAO boots."
- note removed: "2N2222 / S8050: flat face to you, legs down = E B C (check yours)."
- note removed: "= higher reading on D1."
- note removed: "A pin driven LOW turns its colour ON."
- note removed: "Below 40% of the start level"
- note removed: "Charge through the XIAO USB-C port."
- note removed: "D0-D5 are ADC1 pins: safe to read with Wi-Fi on."
- note removed: "D2 is a boot strapping pin: the 10k pull-down keeps it low."
- note removed: "Dome facing you, legs down: OUT GND VS."
- note removed: "If boot misbehaves, move the speaker to D8 (GPIO7)."
- note removed: "Longest leg is the common anode: it goes to 3V3."
- note removed: "More light = lower LDR resistance"
- note removed: "Never paint over the dome."
- note removed: "R101"
- note removed: "R108 R109"
- note removed: "Red has a higher resistor because it is brighter."
- note removed: "Room light ~900, covered ~100."
- note removed: "Small speaker, 8 ohm 1 W (TR-WS-2014B)"
- note removed: "Switch sits in the battery + lead."
- note removed: "Teal = waiting, blue = hiding, red = caught,"
- note removed: "The 5V pin is dead on battery, so"
- note removed: "VBAT = battery after the switch,"
- note removed: "Wire and test each block on USB first, fit the battery and switch last."
- note removed: "counts as covered."
- note removed: "loads that need more than 3.3 V use VBAT."
- note removed: "rainbow = survived the round."
- note removed: "to the BAT+ pad under the XIAO."
